File: kicad/dc-motor-control-circuit.kicad_sch (KiCad schematic)
At the start: 0 parts

Commit message: schematic finished
Parts:
- added A1: Arduino Uno R4 WiFi, PCM_arduino-library:Arduino_Uno_R4_WiFi_Shield, symbol arduino-library:Arduino_Uno_R4_WiFi_Shield
- added A2: Adafruit Motor Shield v2.3, Module:Arduino_UNO_R3, symbol arduino-library:Adafruit_MotorShield_v2.3
- added M1, M2: DC Motor, symbol Motor:Motor_DC
- added R1, R2: 200Ω, symbol Device:R_US
- added R_sense (x2): 5000Ω, symbol Device:R_US
- added U1, U2: TCRT5000, tcrt5000:tcrt5000, symbol tcrt5000:TCRT5000
Connections:
- new net: R2.1, U1.A
- new net: A1.A1, A2.10 (A1), R_sense.1, U1.COLL
- new net: A1.A2, A2.11 (A2)
- new net: A1.A3, A2.12 (A3)
- new net: A1.A4, A2.13 (SDA/A4)
- new net: A1.A5, A2.14 (SCL/A5)
- new net: A1.D0 (D0/RX), A2.15 (D0/RX)
- new net: A1.D1 (D1/TX), A2.16 (D1/TX)
- new net: A1.D2, A2.17 (D2)
- new net: A1.D3, A2.18 (D3)
- new net: A1.D4, A2.19 (D4)
- new net: A1.IORF (IOREF), A2.2 (IOREF)
- new net: A1.D5, A2.20 (D5)
- new net: A1.D6, A2.21 (D6)
- new net: A1.D7, A2.22 (D7)
- new net: A1.D8, A2.23 (D8)
- new net: A1.D9, A2.24 (D9)
- new net: A1.D10, A2.25 (D10)
- new net: A1.D11, A2.26 (D11)
- new net: A1.D12, A2.27 (D12)
- new net: A1.D13, A2.28 (D13)
- new net: A1.GND1 (GND), A2.29 (GND)
- new net: A1.RST1 (RESET), A2.3 (~{RESET})
- new net: A1.AREF, A2.30 (AREF)
- new net: A1.SCL, A2.31 (SDA/A4)
- new net: A1.SDA, A2.32 (SCL/A5)
- new net: A2.33 (M1_POS), M1.1 (+)
- new net: A2.34 (M1_NEG), M1.2 (-)
- new net: A2.36 (M2_POS), M2.1 (+)
- new net: A2.37 (M2_NEG), M2.2 (-)
- new net: A1.3V3 (3.3V), A2.4 (3V3)
- new net: A1.GND3 (GND), A2.7 (GND)
- new net: A1.VIN, A2.8 (VIN)
- new net: A1.A0, A2.9 (A0), R_sense.1, U2.COLL
- new net: R1.1, U2.A
- new net +12V: A2.43 (PWR_IN_POS)
- new net +5V: A1.5V1 (5V), A2.5 (+5V), R1.2, R2.2, R_sense.2, R_sense.2
- new net GND: A1.GND2 (GND), A2.44 (POWER_IN_NEG), A2.6 (GND), U1.CATH, U1.E, U2.CATH, U2.E
Other:
- note added: "(Collected from Datasheet)"
- note added: "1mA is typical Collector current for the Phototransistor"
- note added: "5V / 0.001A (1mA) = 5000Ω"
- title: (none) -> DC Motor Control Schematic
